File: PiDriver.kicad_pcb (KiCad board)
At the start: 4 copper layers, 65 x 56 mm, 65 parts, among them J0 Raspberry_Pi_2_3, J1 Screw_Terminal_01x02, J10 Screw_Terminal_01x02, J11 Jack-DC, J12 Screw_Terminal_01x02, J2 Screw_Terminal_01x02, J3 Screw_Terminal_01x02, J4 Screw_Terminal_01x02, J5 Screw_Terminal_01x02, J6 Screw_Terminal_01x02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

Commit message: Removed 5V linear regulator because it generated too much heat.
The 5V linear regulator generated a ton of heat right above the Pi
processor, which caused it to thermally-overload and reset. So, we won't
try to power the Pi from this board for now. In the future, we could use
a more efficient switching supply that wouldn't generate as much heat.
But, we can separately power the Pi via USB for now.
Parts:
- removed C1, C3: 10uF, Capacitor_Tantalum_SMD:CP_EIA-7343-31_Kemet-D_Pad2.25x2.55mm_HandSolder
- removed C2, C4: DNP, Capacitor_SMD:C_0805_2012Metric_Pad1.15x1.40mm_HandSolder
- removed U1: LM1085-5.0, Package_TO_SOT_SMD:TO-263-3_TabPin2
Connections:
- J0 pad 2: +5V -> Net-(J0-Pad2)
- J0 pad 4: +5V -> Net-(J0-Pad4)
Routing:
- net GND: track 63.6 -> 45.7 mm, vias 2 -> 0
- net +5V: track 17.4 -> 0.00 mm
- net VCC: track 70.3 -> 58.9 mm, vias 1 -> 0
- removed copper zone on F.Cu, net +5V
Other:
- board text added: "+-"
- board text added: "PiDRIVER REV: 2"
- board text removed: "PiDRIVER REV: 1"
